File: LED/LED.kicad_sch (KiCad schematic)
At the start: 0 parts

Commit message: feat: add LED png and kicad pcb files
Parts:
- added BT1: Battery, Connector_PinHeader_1.00mm:PinHeader_2x01_P1.00mm_Vertical, symbol Device:Battery
- added D1: LED, LED_THT:LED_D5.0mm, symbol Device:LED
- added R1: R, Resistor_THT:R_Axial_DIN0204_L3.6mm_D1.6mm_P5.08mm_Horizontal, symbol Device:R
Connections:
- new net: BT1.1 (+), R1.1
- new net: BT1.2 (-), D1.1 (K)
- new net: D1.2 (A), R1.2
